File: motor_ctrl.kicad_pcb (KiCad board)
At the start: 2 copper layers, 92 x 76 mm, 59 parts, among them J1 BATTERY 12V, J2 MOTOR, J3 USB-C, J4 AUX, Q1 IPD90P04P4L-04, Q2 IPD90N04S4L-04, SW1 RESET, SW2 BOOT, U1 LMR33630ADDA, U2 UCC27517A, U3 ESP32-S3-WROOM-1, U4 USBLC6-2SC6

Commit message: PCB: clear KiCad DRC errors, tidy silkscreen, fill zones
First run of real KiCad DRC (7.0.11) on the generated board found:
- 8 clearance errors inside the USB-C footprint (VBUS/GND pads are
  0.2 mm apart by design vs 0.25 mm Supply class): J3 footprint
  clearance override set to 0.2 mm.
- 4 starved thermal reliefs on U1's exposed-pad vias: U1 footprint
  zone connection set to solid (also better for heat).
- Dangling V12 track on B.Cu under D3's top-only tab: bottom copy now
  starts at the first stitching via.
- Silkscreen overlaps/edge clipping: new place_refs.py moves reference
  designators to clean spots; mounting-hole refs hidden; J4 pin labels
  split per pin at 0.8 mm (min text height).

Also: fplib.py paths come from KICAD_FP_DIR / ESP_FP_DIR; ESP32 antenna
keepout written with explicit F.Cu+B.Cu layers; kicad_finish.py fills
zones and writes the DRC report. The delivered board is now zone-filled.

Remaining DRC items: 4 silk warnings from L1's own library footprint
arcs. 0 unconnected pads, 0 copper/clearance/courtyard errors.

Co-Authored-By: Claude Opus 5.5 <noreply@anthropic.com>
Claude-Session: https://claude.ai/code/session_01PLwf3QU8QPKZDxUzVMVmef
Routing:
- net V12: track 199.5 -> 196.8 mm
Other:
- rule pad_to_mask_clearance: 0.0 -> 0
- board text added: "3V3"
- board text added: "IO5"
- board text added: "IO6"
- board text removed: "3V3 IO5 IO6 GND"

Commit message: Add wiper park-switch input (J5 -> IO7)
The user drives a windscreen wiper motor and wants the blades parked
during pauses, so the motor's park contact needs an input.

- J5 (Phoenix PT 1,5 3.5 mm, 2-pin): 1 = PARK, 2 = GND.
- R17 4k7 (1206) pulls PARK up to V12: open contact reads 12 V and
  the cam contact gets ~3 mA of wetting current.
- R18 100k / R19 10k scale PARK by 1/11, so a 32 V load dump gives
  2.9 V at the pin; no clamp needed. C18 470 nF (tau 4.3 ms) removes
  the 20 kHz ripple a 31b-style park contact sees through MOTOR_N.
- PARK_ADC goes to U3 pin 7 = IO7 (ADC1_CH6).

PCB: parts placed below the module, routed by the new route_extra.py
(two-layer grid A* that leaves the frozen routing untouched; it removed
4 GND stitching vias that sat on the new copper). place_refs.py now
deletes footprint silk arcs that overlap a pad (J5, L1), keeping lines
that only come close (diode cathode marks). KiCad DRC: clean, 0
unconnected. ERC 0/0. Netlist vs board: 64/64 parts, 32/32 nets.
BOM regenerated (make_bom.py takes an output path).

Co-Authored-By: Claude Opus 5.5 <noreply@anthropic.com>
Claude-Session: https://claude.ai/code/session_01PLwf3QU8QPKZDxUzVMVmef
Parts:
- added C18: 470nF, Capacitor_SMD:C_0805_2012Metric, F.Cu at (154.0, 133.0)
- added J5: PARK, TerminalBlock_Phoenix:TerminalBlock_Phoenix_PT-1,5-2-3.5-H_1x02_P3.50mm_Horizontal, F.Cu at (161.0, 131.4)
- added R17: 4k7, Resistor_SMD:R_1206_3216Metric, F.Cu at (168.5, 134.6)
- added R18: 100k, Resistor_SMD:R_0805_2012Metric, F.Cu at (154.0, 128.2)
- added R19: 10k, Resistor_SMD:R_0805_2012Metric, F.Cu at (154.0, 130.6)
Connections:
- U3 pad 7: (no net) -> PARK_ADC
Routing:
- net PARK_ADC: track 0.00 -> 17.8 mm, vias 0 -> 2
- net PARK: track 0.00 -> 11.3 mm
- net GND: vias 147 -> 143
