File: motor_ctrl.kicad_sch (KiCad schematic)
At the start: 59 parts, among them J1 BATTERY 12V, J2 MOTOR, J3 USB-C, J4 AUX, Q1 IPD90P04P4L-04, Q2 IPD90N04S4L-04, SW1 RESET, SW2 BOOT, U1 LMR33630ADDA, U2 UCC27517A, U3 ESP32-S3-WROOM-1, U4 USBLC6-2SC6

Commit message: Schematic: KiCad 7 format, ERC clean, linked to the board
- gen_sch.py writes the KiCad 7 file format (20230121), which KiCad 7,
  8 and 9 all open; the KiCad 8 format could not be read by KiCad 7.
- Real KiCad ERC (eeschema 7.0.11) first reported 4 "power input not
  driven" errors (VIN_BUCK, GND, VDRV, +3V3: all fed through passive
  parts). Added PWR_FLAGs on those nets. ERC is now 0 errors, 0
  warnings.
- The generated symbols are also written to motor_ctrl.kicad_sym with a
  project sym-lib-table, so the motor_ctrl library resolves and the
  symbols are editable.
- Symbol UUIDs derive from the reference (design.sym_uuid) and
  build_pcb.py writes them as footprint paths, so KiCad links each
  footprint to its symbol. All schematic UUIDs are now deterministic.
- Readability: ref/value of vertical two-pin parts written vertically,
  stacked same-net pairs joined by a wire, adjacent GND pins share one
  GND symbol, power LED moved, ESP32 frame kept inside the border.
- motor_ctrl_schematic.pdf is now plotted by KiCad.
- New tools: compare_sch_pcb.py (KiCad netlist vs board: nets, values,
  footprints, links) and run_erc_gui.sh (headless ERC for KiCad 7).

Co-Authored-By: Claude Opus 5.5 <noreply@anthropic.com>
Claude-Session: https://claude.ai/code/session_01PLwf3QU8QPKZDxUzVMVmef
Other:
- note added: "PWR_FLAG: these nets are fed through passive parts (diodes, R4, L1, J1), so ERC needs a flag"

Commit message: Add wiper park-switch input (J5 -> IO7)
The user drives a windscreen wiper motor and wants the blades parked
during pauses, so the motor's park contact needs an input.

- J5 (Phoenix PT 1,5 3.5 mm, 2-pin): 1 = PARK, 2 = GND.
- R17 4k7 (1206) pulls PARK up to V12: open contact reads 12 V and
  the cam contact gets ~3 mA of wetting current.
- R18 100k / R19 10k scale PARK by 1/11, so a 32 V load dump gives
  2.9 V at the pin; no clamp needed. C18 470 nF (tau 4.3 ms) removes
  the 20 kHz ripple a 31b-style park contact sees through MOTOR_N.
- PARK_ADC goes to U3 pin 7 = IO7 (ADC1_CH6).

PCB: parts placed below the module, routed by the new route_extra.py
(two-layer grid A* that leaves the frozen routing untouched; it removed
4 GND stitching vias that sat on the new copper). place_refs.py now
deletes footprint silk arcs that overlap a pad (J5, L1), keeping lines
that only come close (diode cathode marks). KiCad DRC: clean, 0
unconnected. ERC 0/0. Netlist vs board: 64/64 parts, 32/32 nets.
BOM regenerated (make_bom.py takes an output path).

Co-Authored-By: Claude Opus 5.5 <noreply@anthropic.com>
Claude-Session: https://claude.ai/code/session_01PLwf3QU8QPKZDxUzVMVmef
Parts:
- added C18: 470nF, Capacitor_SMD:C_0805_2012Metric, symbol motor_ctrl:c
- added J5: PARK, TerminalBlock_Phoenix:TerminalBlock_Phoenix_PT-1,5-2-3.5-H_1x02_P3.50mm_Horizontal, symbol motor_ctrl:conn2
- added R17: 4k7, Resistor_SMD:R_1206_3216Metric, symbol motor_ctrl:r
- added R18: 100k, Resistor_SMD:R_0805_2012Metric, symbol motor_ctrl:r
- added R19: 10k, Resistor_SMD:R_0805_2012Metric, symbol motor_ctrl:r
Connections:
- net GND: now also C18.2, J5.2 (Pin_2), R19.2
- net V12: now also R17.1
- net PARK_ADC: now reaches U3.7 (IO7)
- net PARK_ADC: now also C18.1, R18.2, R19.1
- new net PARK: J5.1 (Pin_1), R17.2, R18.1
- no-connect marks 31 -> 30
Other:
- note added: "J5 park input: IO7 reads PARK / 11. Firmware compares it with the battery voltage (works for contact-to-GND and 31b park switches)."
- note added: "WIPER PARK SWITCH INPUT"
